File: HARDWARE/EDA/KICAD/pswclsx6socket/pswclsx6socket.kicad_pcb (KiCad board)
At the start: 2 copper layers, 115 x 21.8 mm, 7 parts, among them J1 pswcls-master, J2 pswcls-1, J3 pswcls-2, J4 pswcls-3, J5 pswcls-4, J6 pswcls-5, J7 pswcls-6

Commit message: complement adjusts
Parts:
- removed the J1 at (93.1, 89.8)
- removed the J2 at (111.1, 94.8)
- removed the J3 at (129.1, 94.8)
- removed the J4 at (147.1, 94.8)
- removed the J5 at (165.1, 94.8)
- removed the J6 at (183.1, 94.8)
- removed the J7 at (201.1, 94.8)
- added J1: pswcls-master, Connector_PinSocket_2.54mm:PinSocket_1x08_P2.54mm_Vertical, F.Cu at (272.9, 103.9)
- added J1: pswcls-master, Connector_PinSocket_2.54mm:PinSocket_1x08_P2.54mm_Vertical, F.Cu at (272.9, 68.9)
- added J1: pswcls-master, Connector_PinSocket_2.54mm:PinSocket_1x08_P2.54mm_Vertical, F.Cu at (272.9, 138.9)
- added J1: pswcls-master, Connector_PinSocket_2.54mm:PinSocket_1x08_P2.54mm_Vertical, F.Cu at (272.9, 33.9)
- added J1: pswcls-master, Connector_PinSocket_2.54mm:PinSocket_1x08_P2.54mm_Vertical, F.Cu at (142.9, 33.9)
- added J1: pswcls-master, Connector_PinSocket_2.54mm:PinSocket_1x08_P2.54mm_Vertical, F.Cu at (142.9, 68.9)
- added J1: pswcls-master, Connector_PinSocket_2.54mm:PinSocket_1x08_P2.54mm_Vertical, F.Cu at (142.9, 103.9)
- added J1: pswcls-master, Connector_PinSocket_2.54mm:PinSocket_1x08_P2.54mm_Vertical, F.Cu at (142.9, 138.9)
- added J1: pswcls-master, Connector_PinSocket_2.54mm:PinSocket_1x08_P2.54mm_Vertical, F.Cu at (142.9, 173.9)
- added J2: pswcls-1, Connector_PinSocket_2.54mm:PinSocket_1x03_P2.54mm_Vertical, F.Cu at (164.9, 103.9)
- added J2: pswcls-1, Connector_PinSocket_2.54mm:PinSocket_1x03_P2.54mm_Vertical, F.Cu at (164.9, 138.9)
- added J2: pswcls-1, Connector_PinSocket_2.54mm:PinSocket_1x03_P2.54mm_Vertical, F.Cu at (164.9, 33.9)
- added J2: pswcls-1, Connector_PinSocket_2.54mm:PinSocket_1x03_P2.54mm_Vertical, F.Cu at (164.9, 68.9)
- added J2: pswcls-1, Connector_PinSocket_2.54mm:PinSocket_1x03_P2.54mm_Vertical, F.Cu at (34.9, 33.9)
- added J2: pswcls-1, Connector_PinSocket_2.54mm:PinSocket_1x03_P2.54mm_Vertical, F.Cu at (34.9, 68.9)
- added J2: pswcls-1, Connector_PinSocket_2.54mm:PinSocket_1x03_P2.54mm_Vertical, F.Cu at (34.9, 103.9)
- added J2: pswcls-1, Connector_PinSocket_2.54mm:PinSocket_1x03_P2.54mm_Vertical, F.Cu at (34.9, 138.9)
- added J2: pswcls-1, Connector_PinSocket_2.54mm:PinSocket_1x03_P2.54mm_Vertical, F.Cu at (34.9, 173.9)
- added J3: pswcls-2, Connector_PinSocket_2.54mm:PinSocket_1x03_P2.54mm_Vertical, F.Cu at (182.9, 68.9)
- added J3: pswcls-2, Connector_PinSocket_2.54mm:PinSocket_1x03_P2.54mm_Vertical, F.Cu at (182.9, 33.9)
- added J3: pswcls-2, Connector_PinSocket_2.54mm:PinSocket_1x03_P2.54mm_Vertical, F.Cu at (182.9, 138.9)
- added J3: pswcls-2, Connector_PinSocket_2.54mm:PinSocket_1x03_P2.54mm_Vertical, F.Cu at (182.9, 103.9)
- added J3: pswcls-2, Connector_PinSocket_2.54mm:PinSocket_1x03_P2.54mm_Vertical, F.Cu at (52.9, 33.9)
- added J3: pswcls-2, Connector_PinSocket_2.54mm:PinSocket_1x03_P2.54mm_Vertical, F.Cu at (52.9, 68.9)
- added J3: pswcls-2, Connector_PinSocket_2.54mm:PinSocket_1x03_P2.54mm_Vertical, F.Cu at (52.9, 103.9)
- added J3: pswcls-2, Connector_PinSocket_2.54mm:PinSocket_1x03_P2.54mm_Vertical, F.Cu at (52.9, 138.9)
- added J3: pswcls-2, Connector_PinSocket_2.54mm:PinSocket_1x03_P2.54mm_Vertical, F.Cu at (52.9, 173.9)
- added J4: pswcls-3, Connector_PinSocket_2.54mm:PinSocket_1x03_P2.54mm_Vertical, F.Cu at (200.9, 138.9)
- added J4: pswcls-3, Connector_PinSocket_2.54mm:PinSocket_1x03_P2.54mm_Vertical, F.Cu at (200.9, 33.9)
- added J4: pswcls-3, Connector_PinSocket_2.54mm:PinSocket_1x03_P2.54mm_Vertical, F.Cu at (200.9, 68.9)
- added J4: pswcls-3, Connector_PinSocket_2.54mm:PinSocket_1x03_P2.54mm_Vertical, F.Cu at (200.9, 103.9)
- added J4: pswcls-3, Connector_PinSocket_2.54mm:PinSocket_1x03_P2.54mm_Vertical, F.Cu at (70.9, 33.9)
- added J4: pswcls-3, Connector_PinSocket_2.54mm:PinSocket_1x03_P2.54mm_Vertical, F.Cu at (70.9, 68.9)
- added J4: pswcls-3, Connector_PinSocket_2.54mm:PinSocket_1x03_P2.54mm_Vertical, F.Cu at (70.9, 103.9)
- added J4: pswcls-3, Connector_PinSocket_2.54mm:PinSocket_1x03_P2.54mm_Vertical, F.Cu at (70.9, 138.9)
- added J4: pswcls-3, Connector_PinSocket_2.54mm:PinSocket_1x03_P2.54mm_Vertical, F.Cu at (70.9, 173.9)
- added J5: pswcls-4, Connector_PinSocket_2.54mm:PinSocket_1x03_P2.54mm_Vertical, F.Cu at (218.9, 138.9)
- added J5: pswcls-4, Connector_PinSocket_2.54mm:PinSocket_1x03_P2.54mm_Vertical, F.Cu at (218.9, 103.9)
- added J5: pswcls-4, Connector_PinSocket_2.54mm:PinSocket_1x03_P2.54mm_Vertical, F.Cu at (218.9, 33.9)
- added J5: pswcls-4, Connector_PinSocket_2.54mm:PinSocket_1x03_P2.54mm_Vertical, F.Cu at (218.9, 68.9)
- added J5: pswcls-4, Connector_PinSocket_2.54mm:PinSocket_1x03_P2.54mm_Vertical, F.Cu at (88.9, 33.9)
- added J5: pswcls-4, Connector_PinSocket_2.54mm:PinSocket_1x03_P2.54mm_Vertical, F.Cu at (88.9, 68.9)
- added J5: pswcls-4, Connector_PinSocket_2.54mm:PinSocket_1x03_P2.54mm_Vertical, F.Cu at (88.9, 103.9)
- added J5: pswcls-4, Connector_PinSocket_2.54mm:PinSocket_1x03_P2.54mm_Vertical, F.Cu at (88.9, 138.9)
- added J5: pswcls-4, Connector_PinSocket_2.54mm:PinSocket_1x03_P2.54mm_Vertical, F.Cu at (88.9, 173.9)
- added J6: pswcls-5, Connector_PinSocket_2.54mm:PinSocket_1x03_P2.54mm_Vertical, F.Cu at (236.9, 68.9)
- added J6: pswcls-5, Connector_PinSocket_2.54mm:PinSocket_1x03_P2.54mm_Vertical, F.Cu at (236.9, 33.9)
- added J6: pswcls-5, Connector_PinSocket_2.54mm:PinSocket_1x03_P2.54mm_Vertical, F.Cu at (236.9, 138.9)
- added J6: pswcls-5, Connector_PinSocket_2.54mm:PinSocket_1x03_P2.54mm_Vertical, F.Cu at (236.9, 103.9)
- added J6: pswcls-5, Connector_PinSocket_2.54mm:PinSocket_1x03_P2.54mm_Vertical, F.Cu at (106.9, 33.9)
- added J6: pswcls-5, Connector_PinSocket_2.54mm:PinSocket_1x03_P2.54mm_Vertical, F.Cu at (106.9, 68.9)
- added J6: pswcls-5, Connector_PinSocket_2.54mm:PinSocket_1x03_P2.54mm_Vertical, F.Cu at (106.9, 103.9)
- added J6: pswcls-5, Connector_PinSocket_2.54mm:PinSocket_1x03_P2.54mm_Vertical, F.Cu at (106.9, 138.9)
- added J6: pswcls-5, Connector_PinSocket_2.54mm:PinSocket_1x03_P2.54mm_Vertical, F.Cu at (106.9, 173.9)
- added J7: pswcls-6, Connector_PinSocket_2.54mm:PinSocket_1x03_P2.54mm_Vertical, F.Cu at (254.9, 68.9)
- added J7: pswcls-6, Connector_PinSocket_2.54mm:PinSocket_1x03_P2.54mm_Vertical, F.Cu at (254.9, 33.9)
- added J7: pswcls-6, Connector_PinSocket_2.54mm:PinSocket_1x03_P2.54mm_Vertical, F.Cu at (254.9, 138.9)
- added J7: pswcls-6, Connector_PinSocket_2.54mm:PinSocket_1x03_P2.54mm_Vertical, F.Cu at (254.9, 103.9)
- added J7: pswcls-6, Connector_PinSocket_2.54mm:PinSocket_1x03_P2.54mm_Vertical, F.Cu at (124.9, 33.9)
- added J7: pswcls-6, Connector_PinSocket_2.54mm:PinSocket_1x03_P2.54mm_Vertical, F.Cu at (124.9, 68.9)
- added J7: pswcls-6, Connector_PinSocket_2.54mm:PinSocket_1x03_P2.54mm_Vertical, F.Cu at (124.9, 103.9)
- added J7: pswcls-6, Connector_PinSocket_2.54mm:PinSocket_1x03_P2.54mm_Vertical, F.Cu at (124.9, 138.9)
- added J7: pswcls-6, Connector_PinSocket_2.54mm:PinSocket_1x03_P2.54mm_Vertical, F.Cu at (124.9, 173.9)
Routing:
- net (no net): track 0.00 -> 5489.2 mm
- net vll_relay-6: track 119.8 -> 0.00 mm, vias 2 -> 0
- net GND: track 110.1 -> 0.00 mm
- net vcc_relay-master: track 108.0 -> 0.00 mm, vias 2 -> 0
- net vll_relay-5: track 100.7 -> 0.00 mm, vias 2 -> 0
- net vll_relay-4: track 81.7 -> 0.00 mm, vias 2 -> 0
- net vll_relay-3: track 63.3 -> 0.00 mm, vias 2 -> 0
- net vll_relay-2: track 44.7 -> 0.00 mm, vias 2 -> 0
- net vll_relay-1: track 26.2 -> 0.00 mm, vias 2 -> 0
Other:
- board size 115 x 21.8 mm -> 244.1 x 160.4 mm
