File: HARDWARE/EDA/KICAD/pswclsx6socket/pswclsx6socket.sch (KiCad schematic (older format))
At the start: 7 parts, among them J1 pswcls-master, J2 pswcls-1, J3 pswcls-2, J4 pswcls-3, J5 pswcls-4, J6 pswcls-5, J7 pswcls-6

Commit message: complement adjusts
Connections:
- net vll_relay-1: now also J1.8 (Pin_8); no longer J1.3 (Pin_3)
- net vll_relay-2: now also J1.7 (Pin_7); no longer J1.4 (Pin_4)
- net vll_relay-3: now also J1.6 (Pin_6); no longer J1.5 (Pin_5)
- net vll_relay-4: now also J1.5 (Pin_5); no longer J1.6 (Pin_6)
- net vll_relay-5: now also J1.4 (Pin_4); no longer J1.7 (Pin_7)
- net vll_relay-6: now also J1.3 (Pin_3); no longer J1.8 (Pin_8)
Other:
- moved on the sheet: J1, J2, J3, J4, J5, J6, J7
